File: privat/analog_supply_V1.0/analog_supply_V1.0.kicad_pcb (KiCad board)
At the start: 2 copper layers, 111 x 54 mm, 39 parts, among them J1 Screw_Terminal_01x02, J2 Screw_Terminal_01x02, J3 Screw_Terminal_01x03, U1 LM317_TO-220, U2 LM317_TO-220, U3 LM337_TO220, U4 LM337_TO220, X2 PN87520

Commit message: analog_supply_V1.0 add order numbers
Parts:
- H1, H2, H3, H4: footprint MountingHole:MountingHole_3.2mm_M3_DIN965_Pad_TopBottom -> MountingHole:MountingHole_3.2mm_M3_DIN965_Pad
- R1, R5: value 47K -> 750R
- R2, R6: value 47K -> 2K2
- R3, R4, R7, R8: value 47K -> 240R

Commit message: neu: LM2575Mod_V1.1 ESP12E-rolladen_V1.0 ESP12E-rolladen(V1.1)
Parts:
- B1: value KBU4G DIO -> KBU4G
- C10, C11, C15, C16, C3, C4, C5, C9: value X7R-5 100N -> X7R-G1206 100N
- J1: value Screw_Terminal_01x02 -> AKL 171-2
- J2: value Screw_Terminal_01x02 -> AKL 101-2
- J3: value Screw_Terminal_01x03 -> AKL 101-3
