File: privat/analog_supply_V1.0/analog_supply_V1.0.sch (KiCad schematic (older format))
At the start: 39 parts, among them J1 Screw_Terminal_01x02, J2 Screw_Terminal_01x02, J3 Screw_Terminal_01x03, U1 LM317_TO-220, U2 LM317_TO-220, U3 LM337_TO220, U4 LM337_TO220, X2 PN87520

Commit message: analog_supply_V1.0 add order numbers
Parts:
- B1: Bestellnummer (none) -> KBU4G DIO
- C1, C8: Bestellnummer (none) -> RAD FC 470/35
- C10, C11, C15, C16, C3, C4, C5, C9: Bestellnummer (none) -> X7R-5 100N
- C12, C17, C18, C2: Bestellnummer (none) -> RAD LXZ 16/1K0
- H1, H2, H3, H4: footprint MountingHole:MountingHole_3.2mm_M3_DIN965_Pad_TopBottom -> MountingHole:MountingHole_3.2mm_M3_DIN965_Pad
- R1, R5: value 47K -> 750R; Bestellnummer (none) -> SMD 1/4W 750
- R2, R6: value 47K -> 2K2; Bestellnummer (none) -> SMD 1/4W 1,5K
- R3, R4, R7, R8: value 47K -> 240R; Bestellnummer (none) -> SMD 1/4W 240
- TR1: Bestellnummer (none) -> EI 48/16,8 212
- U1, U2: Bestellnummer (none) -> LM 317-220
- U3, U4: Bestellnummer (none) -> LM 337-220
Changed lines of the file:
@@
 F 2 "analog_supply_V1.0:E5-8,5" H 5800 3100 50  0001 C CNN
 F 3 "" H 5800 3100 50  0001 C CNN
+F 4 "RAD FC 470/35" H 5800 3100 50  0001 C CNN "Bestellnummer"
 	1    5800 3100
 	1    0    0    -1
@@
 F 2 "analog_supply_V1.0:E5-8,5" H 7950 1750 50  0001 C CNN
 F 3 "" H 7950 1750 50  0001 C CNN
+F 4 "RAD LXZ 16/1K0" H 7950 1750 50  0001 C CNN "Bestellnummer"
 	1    7950 1750
 	1    0    0    -1
@@
 F 2 "Capacitor_SMD:C_1206_3216Metric_Pad1.33x1.80mm_HandSolder" H 6000 3100 50  0001 C CNN
 F 3 "" H 6000 3100 50  0001 C CNN
+F 4 "X7R-5 100N" H 6000 3100 50  0001 C CNN "Bestellnummer"
 	1    6000 3100
 	1    0    0    -1
@@
 F 2 "Capacitor_SMD:C_1206_3216Metric_Pad1.33x1.80mm_HandSolder" H 7750 1750 50  0001 C CNN
 F 3 "" H 7750 1750 50  0001 C CNN
+F 4 "X7R-5 100N" H 7750 1750 50  0001 C CNN "Bestellnummer"
 	1    7750 1750
 	1    0    0    -1
@@
 F 2 "Capacitor_SMD:C_1206_3216Metric_Pad1.33x1.80mm_HandSolder" H 6200 3100 50  0001 C CNN
 F 3 "" H 6200 3100 50  0001 C CNN
+F 4 "X7R-5 100N" H 6200 3100 50  0001 C CNN "Bestellnummer"
 	1    6200 3100
 	1    0    0    -1
@@
 F 2 "analog_supply_V1.0:KBU" H 4900 2800 50  0001 C CNN
 F 3 "" H 4900 2800 50  0001 C CNN
+F 4 "KBU4G DIO" H 4900 2800 50  0001 C CNN "Bestellnummer"
 	1    4900 2800
 	1    0    0    1
@@
 F 2 "analog_supply_V1.0:EI48-1" H 3600 2800 50  0001 C CNN
 F 3 "" H 3600 2800 50  0001 C CNN
+F 4 "EI 48/16,8 212" H 3600 2800 50  0001 C CNN "Bestellnummer"
 	1    3600 2800
 	1    0    0    -1
@@
 F 2 "analog_supply_V1.0:E5-8,5" H 5800 4350 50  0001 C CNN
 F 3 "" H 5800 4350 50  0001 C CNN
+F 4 "RAD FC 470/35" H 5800 4350 50  0001 C CNN "Bestellnummer"
 	1    5800 4350
 	1    0    0    -1
@@
 F 2 "Capacitor_SMD:C_1206_3216Metric_Pad1.33x1.80mm_HandSolder" H 6000 4350 50  0001 C CNN
 F 3 "" H 6000 4350 50  0001 C CNN
+F 4 "X7R-5 100N" H 6000 4350 50  0001 C CNN "Bestellnummer"
 	1    6000 4350
 	1    0    0    -1
@@
 F 2 "Capacitor_SMD:C_1206_3216Metric_Pad1.33x1.80mm_HandSolder" H 6200 4350 50  0001 C CNN
 F 3 "" H 6200 4350 50  0001 C CNN
+F 4 "X7R-5 100N" H 6200 4350 50  0001 C CNN "Bestellnummer"
 	1    6200 4350
 	1    0    0    -1
@@
 P 6650 1600
 F 0 "R1" H 6500 1659 59  0000 L BNN
-F 1 "47K" H 6500 1470 59  0000 L BNN
+F 1 "750R" H 6500 1470 59  0000 L BNN
 F 2 "Resistor_SMD:R_1206_3216Metric_Pad1.30x1.75mm_HandSolder" H 6650 1600 50  0001 C CNN
 F 3 "" H 6650 1600 50  0001 C CNN
+F 4 "SMD 1/4W 750" H 6650 1600 50  0001 C CNN "Bestellnummer"
 	1    6650 1600
 	0    -1   -1   0
@@
 P 7150 1200
 F 0 "R3" H 7000 1259 59  0000 L BNN
-F 1 "47K" H 7000 1070 59  0000 L BNN
+F 1 "240R" H 7000 1070 59  0000 L BNN
 F 2 "Resistor_SMD:R_1206_3216Metric_Pad1.30x1.75mm_HandSolder" H 7150 1200 50  0001 C CNN
 F 3 "" H 7150 1200 50  0001 C CNN
+F 4 "SMD 1/4W 240" H 7150 1200 50  0001 C CNN "Bestellnummer"
 	1    7150 1200
 	0    -1   -1   0
@@
 F 2 "analog_supply_V1.0:E5-8,5" H 7950 3100 50  0001 C CNN
 F 3 "" H 7950 3100 50  0001 C CNN
+F 4 "RAD LXZ 16/1K0" H 7950 3100 50  0001 C CNN "Bestellnummer"
 	1    7950 3100
 	1    0    0    -1
@@
 F 2 "Capacitor_SMD:C_1206_3216Metric_Pad1.33x1.80mm_HandSolder" H 7750 3100 50  0001 C CNN
 F 3 "" H 7750 3100 50  0001 C CNN
+F 4 "X7R-5 100N" H 7750 3100 50  0001 C CNN "Bestellnummer"
 	1    7750 3100
 	1    0    0    -1
@@
 F 2 "Package_TO_SOT_THT:TO-220-3_Vertical" H 6650 2600 50  0001 C CIN
 F 3 "http://www.ti.com/lit/ds/symlink/lm317.pdf" H 6650 2350 50  0001 C CNN
+F 4 "LM 317-220" H 6650 2350 50  0001 C CNN "Bestellnummer"
 	1    6650 2350
 	1    0    0    -1
@@
 P 6650 2950
 F 0 "R2" H 6500 3009 59  0000 L BNN
-F 1 "47K" H 6500 2820 59  0000 L BNN
+F 1 "2K2" H 6500 2820 59  0000 L BNN
 F 2 "Resistor_SMD:R_1206_3216Metric_Pad1.30x1.75mm_HandSolder" H 6650 2950 50  0001 C CNN
 F 3 "" H 6650 2950 50  0001 C CNN
+F 4 "SMD 1/4W 1,5K" H 6650 2950 50  0001 C CNN "Bestellnummer"
 	1    6650 2950
 	0    -1   -1   0
@@
 P 7150 2550
 F 0 "R4" H 7000 2609 59  0000 L BNN
-F 1 "47K" H 7000 2420 59  0000 L BNN
+F 1 "240R" H 7000 2420 59  0000 L BNN
 F 2 "Resistor_SMD:R_1206_3216Metric_Pad1.30x1.75mm_HandSolder" H 7150 2550 50  0001 C CNN
 F 3 "" H 7150 2550 50  0001 C CNN
+F 4 "SMD 1/4W 240" H 7150 2550 50  0001 C CNN "Bestellnummer"
 	1    7150 2550
 	0    -1   -1   0
@@
 F 2 "Package_TO_SOT_THT:TO-220-3_Vertical" H 6650 1250 50  0001 C CIN
 F 3 "http://www.ti.com/lit/ds/symlink/lm317.pdf" H 6650 1000 50  0001 C CNN
+F 4 "LM 317-220" H 6650 1000 50  0001 C CNN "Bestellnummer"
 	1    6650 1000
 	1    0    0    -1
@@
 F 2 "Package_TO_SOT_THT:TO-220-3_Vertical" H 6650 4450 50  0001 C CIN
 F 3 "http://www.ti.com/lit/ds/symlink/lm337-n.pdf" H 6650 4650 50  0001 C CNN
+F 4 "LM 337-220" H 6650 4650 50  0001 C CNN "Bestellnummer"
 	1    6650 4650
 	1    0    0    -1
@@
 P 6650 4050
 F 0 "R5" H 6500 4109 59  0000 L BNN
-F 1 "47K" H 6500 3920 59  0000 L BNN
+F 1 "750R" H 6500 3920 59  0000 L BNN
 F 2 "Resistor_SMD:R_1206_3216Metric_Pad1.30x1.75mm_HandSolder" H 6650 4050 50  0001 C CNN
 F 3 "" H 6650 4050 50  0001 C CNN
+F 4 "SMD 1/4W 750" H 6650 4050 50  0001 C CNN "Bestellnummer"
 	1    6650 4050
 	0    -1   1    0
@@
 P 7150 4450
 F 0 "R7" H 7000 4509 59  0000 L BNN
-F 1 "47K" H 7000 4320 59  0000 L BNN
+F 1 "240R" H 7000 4320 59  0000 L BNN
 F 2 "Resistor_SMD:R_1206_3216Metric_Pad1.30x1.75mm_HandSolder" H 7150 4450 50  0001 C CNN
 F 3 "" H 7150 4450 50  0001 C CNN
+F 4 "SMD 1/4W 240" H 7150 4450 50  0001 C CNN "Bestellnummer"
 	1    7150 4450
 	0    -1   1    0
@@
 F 2 "Package_TO_SOT_THT:TO-220-3_Vertical" H 6650 5750 50  0001 C CIN
 F 3 "http://www.ti.com/lit/ds/symlink/lm337-n.pdf" H 6650 5950 50  0001 C CNN
+F 4 "LM 337-220" H 6650 5950 50  0001 C CNN "Bestellnummer"
 	1    6650 5950
 	1    0    0    -1
@@
 P 6650 5350
 F 0 "R6" H 6500 5409 59  0000 L BNN
-F 1 "47K" H 6500 5220 59  0000 L BNN
+F 1 "2K2" H 6500 5220 59  0000 L BNN
 F 2 "Resistor_SMD:R_1206_3216Metric_Pad1.30x1.75mm_HandSolder" H 6650 5350 50  0001 C CNN
 F 3 "" H 6650 5350 50  0001 C CNN
+F 4 "SMD 1/4W 1,5K" H 6650 5350 50  0001 C CNN "Bestellnummer"
 	1    6650 5350
 	0    -1   1    0
@@
 P 7150 5750
 F 0 "R8" H 7000 5809 59  0000 L BNN
-F 1 "47K" H 7000 5620 59  0000 L BNN
+F 1 "240R" H 7000 5620 59  0000 L BNN
 F 2 "Resistor_SMD:R_1206_3216Metric_Pad1.30x1.75mm_HandSolder" H 7150 5750 50  0001 C CNN
 F 3 "" H 7150 5750 50  0001 C CNN
+F 4 "SMD 1/4W 240" H 7150 5750 50  0001 C CNN "Bestellnummer"
 	1    7150 5750
 	0    -1   1    0
@@
 F 2 "analog_supply_V1.0:E5-8,5" H 7950 4350 50  0001 C CNN
 F 3 "" H 7950 4350 50  0001 C CNN
+F 4 "RAD LXZ 16/1K0" H 7950 4350 50  0001 C CNN "Bestellnummer"
 	1    7950 4350
 	1    0    0    -1
@@
 F 2 "Capacitor_SMD:C_1206_3216Metric_Pad1.33x1.80mm_HandSolder" H 7750 4350 50  0001 C CNN
 F 3 "" H 7750 4350 50  0001 C CNN
+F 4 "X7R-5 100N" H 7750 4350 50  0001 C CNN "Bestellnummer"
 	1    7750 4350
 	1    0    0    -1
@@
 F 2 "analog_supply_V1.0:E5-8,5" H 7950 5650 50  0001 C CNN
 F 3 "" H 7950 5650 50  0001 C CNN
+F 4 "RAD LXZ 16/1K0" H 7950 5650 50  0001 C CNN "Bestellnummer"
 	1    7950 5650
 	1    0    0    -1
@@
 F 2 "Capacitor_SMD:C_1206_3216Metric_Pad1.33x1.80mm_HandSolder" H 7750 5650 50  0001 C CNN
 F 3 "" H 7750 5650 50  0001 C CNN
+F 4 "X7R-5 100N" H 7750 5650 50  0001 C CNN "Bestellnummer"
 	1    7750 5650
 	1    0    0    -1
@@
 F 0 "H1" H 3700 5596 50  0000 L CNN
 F 1 "MountingHole" H 3700 5505 50  0000 L CNN
-F 2 "MountingHole:MountingHole_3.2mm_M3_DIN965_Pad_TopBottom" H 3600 5550 50  0001 C CNN
+F 2 "MountingHole:MountingHole_3.2mm_M3_DIN965_Pad" H 3600 5550 50  0001 C CNN
 F 3 "~" H 3600 5550 50  0001 C CNN
 	1    3600 5550
@@
 F 0 "H2" H 3700 5896 50  0000 L CNN
 F 1 "MountingHole" H 3700 5805 50  0000 L CNN
-F 2 "MountingHole:MountingHole_3.2mm_M3_DIN965_Pad_TopBottom" H 3600 5850 50  0001 C CNN
+F 2 "MountingHole:MountingHole_3.2mm_M3_DIN965_Pad" H 3600 5850 50  0001 C CNN
 F 3 "~" H 3600 5850 50  0001 C CNN
 	1    3600 5850
@@
 F 0 "H3" H 3700 6196 50  0000 L CNN
 F 1 "MountingHole" H 3700 6105 50  0000 L CNN
-F 2 "MountingHole:MountingHole_3.2mm_M3_DIN965_Pad_TopBottom" H 3600 6150 50  0001 C CNN
+F 2 "MountingHole:MountingHole_3.2mm_M3_DIN965_Pad" H 3600 6150 50  0001 C CNN
 F 3 "~" H 3600 6150 50  0001 C CNN
 	1    3600 6150
@@
 F 0 "H4" H 3700 6496 50  0000 L CNN
 F 1 "MountingHole" H 3700 6405 50  0000 L CNN
-F 2 "MountingHole:MountingHole_3.2mm_M3_DIN965_Pad_TopBottom" H 3600 6450 50  0001 C CNN
+F 2 "MountingHole:MountingHole_3.2mm_M3_DIN965_Pad" H 3600 6450 50  0001 C CNN
 F 3 "~" H 3600 6450 50  0001 C CNN
 	1    3600 6450

Commit message: neu: LM2575Mod_V1.1 ESP12E-rolladen_V1.0 ESP12E-rolladen(V1.1)
Parts:
- B1: value KBU4G DIO -> KBU4G; Bestellnummer KBU4G DIO -> KBU4G
- C10, C11, C15, C16, C3, C4, C5, C9: value X7R-5 100N -> X7R-G1206 100N; Bestellnummer X7R-5 100N -> X7R-G1206 100N
- J1: value Screw_Terminal_01x02 -> AKL 171-2; Bestellnummer (none) -> AKL 171-2
- J2: value Screw_Terminal_01x02 -> AKL 101-2; Bestellnummer (none) -> AKL 101-2
- J3: value Screw_Terminal_01x03 -> AKL 101-3; Bestellnummer (none) -> AKL 101-3
Changed lines of the file:
@@
 P 6000 3100
 F 0 "C3" H 5860 2915 59  0000 L BNN
-F 1 "X7R-5 100N" V 5985 3160 59  0000 L BNN
+F 1 "X7R-G1206 100N" V 5985 3160 59  0000 L BNN
 F 2 "Capacitor_SMD:C_1206_3216Metric_Pad1.33x1.80mm_HandSolder" H 6000 3100 50  0001 C CNN
 F 3 "" H 6000 3100 50  0001 C CNN
-F 4 "X7R-5 100N" H 6000 3100 50  0001 C CNN "Bestellnummer"
+F 4 "X7R-G1206 100N" H 6000 3100 50  0001 C CNN "Bestellnummer"
 	1    6000 3100
 	1    0    0    -1
@@
 P 7750 1750
 F 0 "C5" H 7610 1565 59  0000 L BNN
-F 1 "X7R-5 100N" V 7735 1810 59  0000 L BNN
+F 1 "X7R-G1206 100N" V 7735 1810 59  0000 L BNN
 F 2 "Capacitor_SMD:C_1206_3216Metric_Pad1.33x1.80mm_HandSolder" H 7750 1750 50  0001 C CNN
 F 3 "" H 7750 1750 50  0001 C CNN
-F 4 "X7R-5 100N" H 7750 1750 50  0001 C CNN "Bestellnummer"
+F 4 "X7R-G1206 100N" H 7750 1750 50  0001 C CNN "Bestellnummer"
 	1    7750 1750
 	1    0    0    -1
@@
 P 6200 3100
 F 0 "C4" H 6190 2985 59  0000 R TNN
-F 1 "X7R-5 100N" V 6185 3160 59  0000 L BNN
+F 1 "X7R-G1206 100N" V 6185 3160 59  0000 L BNN
 F 2 "Capacitor_SMD:C_1206_3216Metric_Pad1.33x1.80mm_HandSolder" H 6200 3100 50  0001 C CNN
 F 3 "" H 6200 3100 50  0001 C CNN
-F 4 "X7R-5 100N" H 6200 3100 50  0001 C CNN "Bestellnummer"
+F 4 "X7R-G1206 100N" H 6200 3100 50  0001 C CNN "Bestellnummer"
 	1    6200 3100
 	1    0    0    -1
@@
 P 4900 2800
 F 0 "B1" H 5000 2900 59  0000 L BNN
-F 1 "KBU4G DIO" H 5000 2650 59  0000 L BNN
+F 1 "KBU4G" H 5000 2650 59  0000 L BNN
 F 2 "analog_supply_V1.0:KBU" H 4900 2800 50  0001 C CNN
 F 3 "" H 4900 2800 50  0001 C CNN
-F 4 "KBU4G DIO" H 4900 2800 50  0001 C CNN "Bestellnummer"
+F 4 "KBU4G" H 4900 2800 50  0001 C CNN "Bestellnummer"
 	1    4900 2800
 	1    0    0    1
@@
 P 6000 4350
 F 0 "C9" H 5860 4165 59  0000 L BNN
-F 1 "X7R-5 100N" V 5985 4410 59  0000 L BNN
+F 1 "X7R-G1206 100N" V 5985 4410 59  0000 L BNN
 F 2 "Capacitor_SMD:C_1206_3216Metric_Pad1.33x1.80mm_HandSolder" H 6000 4350 50  0001 C CNN
 F 3 "" H 6000 4350 50  0001 C CNN
-F 4 "X7R-5 100N" H 6000 4350 50  0001 C CNN "Bestellnummer"
+F 4 "X7R-G1206 100N" H 6000 4350 50  0001 C CNN "Bestellnummer"
 	1    6000 4350
 	1    0    0    -1
@@
 P 6200 4350
 F 0 "C10" H 6190 4235 59  0000 R TNN
-F 1 "X7R-5 100N" V 6185 4410 59  0000 L BNN
+F 1 "X7R-G1206 100N" V 6185 4410 59  0000 L BNN
 F 2 "Capacitor_SMD:C_1206_3216Metric_Pad1.33x1.80mm_HandSolder" H 6200 4350 50  0001 C CNN
 F 3 "" H 6200 4350 50  0001 C CNN
-F 4 "X7R-5 100N" H 6200 4350 50  0001 C CNN "Bestellnummer"
+F 4 "X7R-G1206 100N" H 6200 4350 50  0001 C CNN "Bestellnummer"
 	1    6200 4350
 	1    0    0    -1
@@
 P 7750 3100
 F 0 "C11" H 7610 2915 59  0000 L BNN
-F 1 "X7R-5 100N" V 7735 3160 59  0000 L BNN
+F 1 "X7R-G1206 100N" V 7735 3160 59  0000 L BNN
 F 2 "Capacitor_SMD:C_1206_3216Metric_Pad1.33x1.80mm_HandSolder" H 7750 3100 50  0001 C CNN
 F 3 "" H 7750 3100 50  0001 C CNN
-F 4 "X7R-5 100N" H 7750 3100 50  0001 C CNN "Bestellnummer"
+F 4 "X7R-G1206 100N" H 7750 3100 50  0001 C CNN "Bestellnummer"
 	1    7750 3100
 	1    0    0    -1
@@
 P 1600 2900
 F 0 "J1" H 1518 2575 50  0000 C CNN
-F 1 "Screw_Terminal_01x02" H 1518 2666 50  0000 C CNN
+F 1 "AKL 171-2" H 1518 2666 50  0000 C CNN
 F 2 "TerminalBlock_RND:TerminalBlock_RND_205-00067_1x02_P7.50mm_Horizontal" H 1600 2900 50  0001 C CNN
 F 3 "~" H 1600 2900 50  0001 C CNN
+F 4 "AKL 171-2" H 1600 2900 50  0001 C CNN "Bestellnummer"
 	1    1600 2900
 	-1   0    0    1
@@
 P 7750 4350
 F 0 "C15" H 7610 4165 59  0000 L BNN
-F 1 "X7R-5 100N" V 7735 4410 59  0000 L BNN
+F 1 "X7R-G1206 100N" V 7735 4410 59  0000 L BNN
 F 2 "Capacitor_SMD:C_1206_3216Metric_Pad1.33x1.80mm_HandSolder" H 7750 4350 50  0001 C CNN
 F 3 "" H 7750 4350 50  0001 C CNN
-F 4 "X7R-5 100N" H 7750 4350 50  0001 C CNN "Bestellnummer"
+F 4 "X7R-G1206 100N" H 7750 4350 50  0001 C CNN "Bestellnummer"
 	1    7750 4350
 	1    0    0    -1
@@
 P 7750 5650
 F 0 "C16" H 7610 5465 59  0000 L BNN
-F 1 "X7R-5 100N" V 7735 5710 59  0000 L BNN
+F 1 "X7R-G1206 100N" V 7735 5710 59  0000 L BNN
 F 2 "Capacitor_SMD:C_1206_3216Metric_Pad1.33x1.80mm_HandSolder" H 7750 5650 50  0001 C CNN
 F 3 "" H 7750 5650 50  0001 C CNN
-F 4 "X7R-5 100N" H 7750 5650 50  0001 C CNN "Bestellnummer"
+F 4 "X7R-G1206 100N" H 7750 5650 50  0001 C CNN "Bestellnummer"
 	1    7750 5650
 	1    0    0    -1
@@
 P 9750 2000
 F 0 "J3" H 9830 2042 50  0000 L CNN
-F 1 "Screw_Terminal_01x03" H 9830 1951 50  0000 L CNN
+F 1 "AKL 101-3" H 9830 1951 50  0000 L CNN
 F 2 "TerminalBlock_Phoenix:TerminalBlock_Phoenix_MKDS-1,5-3_1x03_P5.00mm_Horizontal" H 9750 2000 50  0001 C CNN
 F 3 "~" H 9750 2000 50  0001 C CNN
+F 4 "AKL 101-3" H 9750 2000 50  0001 C CNN "Bestellnummer"
 	1    9750 2000
 	1    0    0    -1
@@
 P 9750 1400
 F 0 "J2" H 9830 1392 50  0000 L CNN
-F 1 "Screw_Terminal_01x02" H 9830 1301 50  0000 L CNN
+F 1 "AKL 101-2" H 9830 1301 50  0000 L CNN
 F 2 "TerminalBlock_Phoenix:TerminalBlock_Phoenix_MKDS-1,5-2_1x02_P5.00mm_Horizontal" H 9750 1400 50  0001 C CNN
 F 3 "~" H 9750 1400 50  0001 C CNN
+F 4 "AKL 101-2" H 9750 1400 50  0001 C CNN "Bestellnummer"
 	1    9750 1400
 	1    0    0    -1
