File: pwr_supply_2W/pwr_supply_2W.kicad_pcb (KiCad board)
At the start: 2 copper layers, 80 x 40 mm, 18 parts

Commit message: CP footprint for C103/C104
Parts:
- C104, C?: footprint Capacitor_THT:C_Radial_D8.0mm_H11.5mm_P3.50mm -> Capacitor_THT:CP_Radial_D8.0mm_P3.50mm
Other:
- board text added: "pwr_supply_2W 2022-xx-yy"
- board text removed: "pwr_supply_2W 2022-10-16"
