File: pwr_supply_2W/pwr_supply_2W.kicad_sch (KiCad schematic)
At the start: 18 parts, among them J101 Conn_01x02, J102 Conn_01x02, U101 LM7805_TO220

Commit message: CP footprint for C103/C104
Parts:
- C103, C104: footprint Capacitor_THT:C_Radial_D8.0mm_H11.5mm_P3.50mm -> Capacitor_THT:CP_Radial_D8.0mm_P3.50mm
Changed lines of the file:
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@@
       (effects (font (size 1.27 1.27)) (justify left))
     )
-    (property "Footprint" "Capacitor_THT:C_Radial_D8.0mm_H11.5mm_P3.50mm" (id 2) (at 176.2252 86.36 0)
+    (property "Footprint" "Capacitor_THT:CP_Radial_D8.0mm_P3.50mm" (id 2) (at 176.2252 86.36 0)
       (effects (font (size 1.27 1.27)) hide)
     )
@@
       (effects (font (size 1.27 1.27)) (justify left))
     )
-    (property "Footprint" "Capacitor_THT:C_Radial_D8.0mm_H11.5mm_P3.50mm" (id 2) (at 211.7852 86.36 0)
+    (property "Footprint" "Capacitor_THT:CP_Radial_D8.0mm_P3.50mm" (id 2) (at 211.7852 86.36 0)
       (effects (font (size 1.27 1.27)) hide)
     )
@@
     )
     (path "/a5f783e7-ea52-447e-bc98-90eb5ef612bc"
-      (reference "C103") (unit 1) (value "470uF/25V") (footprint "Capacitor_THT:C_Radial_D8.0mm_H11.5mm_P3.50mm")
+      (reference "C103") (unit 1) (value "470uF/25V") (footprint "Capacitor_THT:CP_Radial_D8.0mm_P3.50mm")
     )
     (path "/c669eb71-27fc-474e-ad66-4f2f275532c7"
-      (reference "C104") (unit 1) (value "470uF/25V") (footprint "Capacitor_THT:C_Radial_D8.0mm_H11.5mm_P3.50mm")
+      (reference "C104") (unit 1) (value "470uF/25V") (footprint "Capacitor_THT:CP_Radial_D8.0mm_P3.50mm")
     )
     (path "/6da15fb6-0bd3-45b0-b831-dbf332c93715"
