File: eload/eload.kicad_pcb (KiCad board)
At the start: 2 copper layers, 49 x 37 mm, 41 parts, among them J101 Conn_01x08, J102 Conn_02x05_Odd_Even, Q101 IRF3205, Q102 IRLIZ44N, Q103 BC847, Q104 BC857, U101 MCP604, U102 OP07

Commit message: eload V1.0 updated measure connections
Connections:
- NT103 pad 2: Net-(NT103-Pad2) -> Net-(U101-Pad3)
- U101 pad 3: Net-(NT102-Pad1) -> Net-(U101-Pad3)
- U101 pad 5: Net-(NT103-Pad2) -> Net-(NT102-Pad1)
Routing:
- net Net-(NT103-Pad2): track 33.8 -> 0.00 mm, vias 2 -> 0
- net Net-(U101-Pad3): track 0.00 -> 33.0 mm, vias 0 -> 2
- net Net-(NT102-Pad1): track 28.7 -> 29.8 mm
Changed lines of the file:
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@@
   (net 35 "/PL0")
   (net 36 "Net-(NT102-Pad1)")
-  (net 37 "Net-(NT103-Pad2)")
+  (net 37 "Net-(U101-Pad3)")
   (footprint "MountingHole:MountingHole_3.2mm_M3_Pad_TopBottom" (layer "F.Cu")
     (at 103.5 53.5)
@@
       (net 4 "Net-(R102-Pad1)") (pinfunction "-") (pintype "input"))
     (pad "3" smd roundrect (at -2.475 -1.27 90) (size 1.95 0.6) (layers "F.Cu" "F.Paste" "F.Mask") (roundrect_rratio 0.25)
-      (net 36 "Net-(NT102-Pad1)") (pinfunction "+") (pintype "input"))
+      (net 37 "Net-(U101-Pad3)") (pinfunction "+") (pintype "input"))
     (pad "4" smd roundrect (at -2.475 0 90) (size 1.95 0.6) (layers "F.Cu" "F.Paste" "F.Mask") (roundrect_rratio 0.25)
       (net 2 "Net-(C101-Pad1)") (pinfunction "V+") (pintype "power_in"))
     (pad "5" smd roundrect (at -2.475 1.27 90) (size 1.95 0.6) (layers "F.Cu" "F.Paste" "F.Mask") (roundrect_rratio 0.25)
-      (net 37 "Net-(NT103-Pad2)") (pinfunction "+") (pintype "input"))
+      (net 36 "Net-(NT102-Pad1)") (pinfunction "+") (pintype "input"))
     (pad "6" smd roundrect (at -2.475 2.54 90) (size 1.95 0.6) (layers "F.Cu" "F.Paste" "F.Mask") (roundrect_rratio 0.25)
       (net 5 "Net-(R102-Pad2)") (pinfunction "-") (pintype "input"))
@@
       (net 33 "/PL2") (pinfunction "1") (pintype "passive"))
     (pad "2" smd circle (at 0.5 0 90) (size 0.5 0.5) (layers "F.Cu")
-      (net 37 "Net-(NT103-Pad2)") (pinfunction "2") (pintype "passive"))
+      (net 37 "Net-(U101-Pad3)") (pinfunction "2") (pintype "passive"))
   )
   (footprint "Resistor_SMD:R_0805_2012Metric_Pad1.20x1.40mm_HandSolder" (layer "F.Cu")
@@
   (segment (start 117.46 84) (end 117.46 83.449085) (width 2) (layer "B.Cu") (net 35))
   (segment (start 111.99952 81.80048) (end 109.7 84.1) (width 2) (layer "B.Cu") (net 35))
-  (segment (start 111.8 78.8) (end 111.8 75.4) (width 0.2) (layer "F.Cu") (net 36))
-  (segment (start 115.8 75.4) (end 111.8 75.4) (width 0.2) (layer "F.Cu") (net 36))
+  (segment (start 111.2 73.3) (end 111.8 73.9) (width 0.2) (layer "F.Cu") (net 36))
+  (segment (start 117.3 73.9) (end 119.5 71.7) (width 0.2) (layer "F.Cu") (net 36))
+  (segment (start 111.8 73.9) (end 117.3 73.9) (width 0.2) (layer "F.Cu") (net 36))
+  (segment (start 111.8 73.9) (end 111.8 78.8) (width 0.2) (layer "F.Cu") (net 36))
   (segment (start 119.065 67.765) (end 119.5 68.2) (width 0.2) (layer "F.Cu") (net 36))
   (segment (start 117.825 67.765) (end 119.065 67.765) (width 0.2) (layer "F.Cu") (net 36))
   (segment (start 119.5 68.2) (end 119.5 71.7) (width 0.2) (layer "F.Cu") (net 36))
-  (segment (start 107.1 70.3) (end 105.93 69.13) (width 0.2) (layer "F.Cu") (net 36))
-  (segment (start 105.93 69.13) (end 105.93 68.375) (width 0.2) (layer "F.Cu") (net 36))
-  (segment (start 107.1 72.9) (end 107.1 70.3) (width 0.2) (layer "F.Cu") (net 36))
-  (segment (start 109.6 75.4) (end 107.1 72.9) (width 0.2) (layer "F.Cu") (net 36))
-  (segment (start 111.8 75.4) (end 109.6 75.4) (width 0.2) (layer "F.Cu") (net 36))
-  (segment (start 119.5 71.7) (end 115.8 75.4) (width 0.2) (layer "F.Cu") (net 36))
-  (segment (start 108.47 68.375) (end 108.47 67.03) (width 0.2) (layer "F.Cu") (net 37))
-  (segment (start 110.41048 67.11048) (end 110.41048 69.81048) (width 0.2) (layer "F.Cu") (net 37))
-  (segment (start 108.47 67.03) (end 108.8 66.7) (width 0.2) (layer "F.Cu") (net 37))
-  (segment (start 108.8 66.7) (end 110 66.7) (width 0.2) (layer "F.Cu") (net 37))
-  (segment (start 110 66.7) (end 110.41048 67.11048) (width 0.2) (layer "F.Cu") (net 37))
-  (segment (start 111.2 73.3) (end 111.8 73.9) (width 0.2) (layer "F.Cu") (net 37))
+  (segment (start 111.2 70.6) (end 111.2 73.3) (width 0.2) (layer "F.Cu") (net 36))
+  (segment (start 110.41048 69.81048) (end 111.2 70.6) (width 0.2) (layer "F.Cu") (net 36))
+  (segment (start 110.41048 67.11048) (end 110.41048 69.81048) (width 0.2) (layer "F.Cu") (net 36))
+  (segment (start 110 66.7) (end 110.41048 67.11048) (width 0.2) (layer "F.Cu") (net 36))
+  (segment (start 108.8 66.7) (end 110 66.7) (width 0.2) (layer "F.Cu") (net 36))
+  (segment (start 108.47 67.03) (end 108.8 66.7) (width 0.2) (layer "F.Cu") (net 36))
+  (segment (start 108.47 68.375) (end 108.47 67.03) (width 0.2) (layer "F.Cu") (net 36))
+  (segment (start 107.1 70.3) (end 105.93 69.13) (width 0.2) (layer "F.Cu") (net 37))
+  (segment (start 105.93 69.13) (end 105.93 68.375) (width 0.2) (layer "F.Cu") (net 37))
+  (segment (start 107.1 72.9) (end 107.1 70.3) (width 0.2) (layer "F.Cu") (net 37))
+  (segment (start 109.6 75.4) (end 110.6 75.4) (width 0.2) (layer "F.Cu") (net 37))
   (segment (start 128 78.1) (end 132.9 78.1) (width 0.2) (layer "F.Cu") (net 37))
-  (segment (start 110.41048 69.81048) (end 111.2 70.6) (width 0.2) (layer "F.Cu") (net 37))
-  (segment (start 111.2 70.6) (end 111.2 73.3) (width 0.2) (layer "F.Cu") (net 37))
-  (segment (start 111.8 73.9) (end 113.8 73.9) (width 0.2) (layer "F.Cu") (net 37))
-  (via (at 113.8 73.9) (size 0.8) (drill 0.4) (layers "F.Cu" "B.Cu") (net 37))
+  (segment (start 109.6 75.4) (end 107.1 72.9) (width 0.2) (layer "F.Cu") (net 37))
+  (via (at 110.6 75.4) (size 0.8) (drill 0.4) (layers "F.Cu" "B.Cu") (net 37))
   (via (at 128 78.1) (size 0.8) (drill 0.4) (layers "F.Cu" "B.Cu") (net 37))
   (segment (start 126.234513 77.534513) (end 126.8 78.1) (width 0.2) (layer "B.Cu") (net 37))
-  (segment (start 113.8 73.9) (end 117.434513 77.534513) (width 0.2) (layer "B.Cu") (net 37))
+  (segment (start 112.734513 77.534513) (end 126.234513 77.534513) (width 0.2) (layer "B.Cu") (net 37))
   (segment (start 126.8 78.1) (end 128 78.1) (width 0.2) (layer "B.Cu") (net 37))
-  (segment (start 117.434513 77.534513) (end 126.234513 77.534513) (width 0.2) (layer "B.Cu") (net 37))
+  (segment (start 110.6 75.4) (end 112.734513 77.534513) (width 0.2) (layer "B.Cu") (net 37))
   (zone (net 13) (net_name "GND") (layer "B.Cu") (hatch edge 0.508)
     (connect_pads (clearance 0.508))
