File: eload/eload.kicad_sch (KiCad schematic)
At the start: 41 parts, among them J101 Conn_01x08, J102 Conn_02x05_Odd_Even, Q101 IRF3205, Q102 IRLIZ44N, Q103 BC847, Q104 BC857, U101 MCP604, U102 OP07

Commit message: eload V1.0 updated measure connections
Connections:
- net at NT103.2: now also U101.3 (+); no longer U101.5 (+)
- net at NT102.1, U102.2 (-): now also U101.5 (+); no longer U101.3 (+)
Changed lines of the file:
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@@
   (junction (at 180.34 113.03) (diameter 0) (color 0 0 0 0)
   )
-  (junction (at 128.27 118.11) (diameter 0) (color 0 0 0 0)
-  )
   (junction (at 212.09 74.93) (diameter 0) (color 0 0 0 0)
   )
   (junction (at 220.98 143.51) (diameter 0) (color 0 0 0 0)
   )
+  (junction (at 128.27 129.54) (diameter 0) (color 0 0 0 0)
+  )
   (junction (at 82.55 154.94) (diameter 0) (color 0 0 0 0)
   )
@@
     (stroke (width 0) (type default) (color 0 0 0 0))
   )
-  (wire (pts (xy 128.27 105.41) (xy 166.37 105.41))
-    (stroke (width 0) (type default) (color 0 0 0 0))
-  )
   (wire (pts (xy 82.55 154.94) (xy 82.55 156.21))
     (stroke (width 0) (type default) (color 0 0 0 0))
@@
     (stroke (width 0) (type default) (color 0 0 0 0))
   )
+  (wire (pts (xy 128.27 163.83) (xy 171.45 163.83))
+    (stroke (width 0) (type default) (color 0 0 0 0))
+  )
   (wire (pts (xy 49.53 125.73) (xy 57.15 125.73))
     (stroke (width 0) (type default) (color 0 0 0 0))
@@
     (stroke (width 0) (type default) (color 0 0 0 0))
   )
-  (wire (pts (xy 166.37 132.08) (xy 166.37 144.78))
-    (stroke (width 0) (type default) (color 0 0 0 0))
-  )
   (wire (pts (xy 212.09 74.93) (xy 212.09 77.47))
     (stroke (width 0) (type default) (color 0 0 0 0))
@@
     (stroke (width 0) (type default) (color 0 0 0 0))
   )
-  (wire (pts (xy 166.37 105.41) (xy 166.37 107.95))
+  (wire (pts (xy 166.37 132.08) (xy 166.37 107.95))
     (stroke (width 0) (type default) (color 0 0 0 0))
   )
@@
     (stroke (width 0) (type default) (color 0 0 0 0))
   )
-  (wire (pts (xy 166.37 144.78) (xy 182.88 144.78))
+  (wire (pts (xy 171.45 144.78) (xy 182.88 144.78))
     (stroke (width 0) (type default) (color 0 0 0 0))
   )
@@
     (stroke (width 0) (type default) (color 0 0 0 0))
   )
+  (wire (pts (xy 171.45 163.83) (xy 171.45 144.78))
+    (stroke (width 0) (type default) (color 0 0 0 0))
+  )
   (wire (pts (xy 90.17 109.22) (xy 90.17 111.76))
     (stroke (width 0) (type default) (color 0 0 0 0))
@@
     (stroke (width 0) (type default) (color 0 0 0 0))
   )
-  (wire (pts (xy 128.27 118.11) (xy 128.27 105.41))
-    (stroke (width 0) (type default) (color 0 0 0 0))
-  )
   (wire (pts (xy 121.92 140.97) (xy 121.92 166.37))
     (stroke (width 0) (type default) (color 0 0 0 0))
@@
     (stroke (width 0) (type default) (color 0 0 0 0))
   )
+  (wire (pts (xy 128.27 129.54) (xy 128.27 163.83))
+    (stroke (width 0) (type default) (color 0 0 0 0))
+  )
